Commit message: Update launch file

File: rm_pioneer_description/urdf/guard.urdf.xacro (robot description, xacro)
@@ -94,3 +94,9 @@
         <axis xyz="0 0 0" />
     </joint>
+    <link name="camera_optical_frame" />
+    <joint name="camera_optical_joint" type="fixed">
+        <origin xyz="0 0 0" rpy="${pi/2} 0 ${pi/2}" />
+        <parent link="camera_base_link" />
+        <child link="camera_optical_frame" />
+    </joint>
 </robot>

File: rm_pioneer_description/urdf/hero.urdf.xacro (robot description, xacro)
@@ -94,3 +94,9 @@
         <axis xyz="0 0 0" />
     </joint>
+    <link name="camera_optical_frame" />
+    <joint name="camera_optical_joint" type="fixed">
+        <origin xyz="0 0 0" rpy="${pi/2} 0 ${pi/2}" />
+        <parent link="camera_base_link" />
+        <child link="camera_optical_frame" />
+    </joint>
 </robot>

Commit message: Fixed a stupid bug

File: rm_pioneer_description/urdf/guard.urdf.xacro (robot description, xacro)
@@ -96,5 +96,5 @@
     <link name="camera_optical_frame" />
     <joint name="camera_optical_joint" type="fixed">
-        <origin xyz="0 0 0" rpy="${pi/2} 0 ${pi/2}" />
+        <origin xyz="0 0 0" rpy="${-pi/2} 0 ${-pi/2}" />
         <parent link="camera_base_link" />
         <child link="camera_optical_frame" />

File: rm_pioneer_description/urdf/hero.urdf.xacro (robot description, xacro)
@@ -96,5 +96,5 @@
     <link name="camera_optical_frame" />
     <joint name="camera_optical_joint" type="fixed">
-        <origin xyz="0 0 0" rpy="${pi/2} 0 ${pi/2}" />
+        <origin xyz="0 0 0" rpy="${-pi/2} 0 ${-pi/2}" />
         <parent link="camera_base_link" />
         <child link="camera_optical_frame" />
