Commit message: Update params for standard5

File: rm_pioneer_description/urdf/standard5.urdf.xacro (robot description, xacro)
@@ -18,5 +18,5 @@
       <origin xyz="0 0 0" rpy="0 0 0" />
       <geometry>
-        <mesh filename="package://rm_pioneer_description/meshes/standard_5/yaw_link.stl" />
+        <mesh filename="package://rm_pioneer_description/meshes/standard5/yaw_link.stl" />
       </geometry>
       <material name="black"/>
@@ -25,5 +25,5 @@
       <origin xyz="0 0 0" rpy="0 0 0" />
       <geometry>
-        <mesh filename="package://rm_pioneer_description/meshes/standard_5/yaw_link.stl" />
+        <mesh filename="package://rm_pioneer_description/meshes/standard5/yaw_link.stl" />
       </geometry>
     </collision>
@@ -44,5 +44,5 @@
       <origin xyz="0 0 0" rpy="0 0 0" />
       <geometry>
-        <mesh filename="package://rm_pioneer_description/meshes/standard_5/pitch_link.stl" />
+        <mesh filename="package://rm_pioneer_description/meshes/standard5/pitch_link.stl" />
       </geometry>
       <material name="gray"/>
@@ -51,5 +51,5 @@
       <origin xyz="0 0 0" rpy="0 0 0" />
       <geometry>
-        <mesh filename="package://rm_pioneer_description/meshes/standard_5/pitch_link.stl" />
+        <mesh filename="package://rm_pioneer_description/meshes/standard5/pitch_link.stl" />
       </geometry>
     </collision>
@@ -59,5 +59,5 @@
     <parent link="yaw_link" />
     <child link="pitch_link" />
-    <axis xyz="0 0 0" />
+    <axis xyz="0 1 0" />
     <limit lower="-0.6" upper="0.5" effort="1.2" velocity="31"/>
   </joint>
@@ -77,5 +77,5 @@
       <origin xyz="0 0 0" rpy="0 0 0" />
       <geometry>
-        <mesh filename="package://rm_pioneer_description/meshes/standard_5/camera_base_link.STL" />
+        <mesh filename="package://rm_pioneer_description/meshes/standard5/camera_base_link.STL" />
       </geometry>
       <material name="cyan">
@@ -86,5 +86,5 @@
       <origin xyz="0 0 0" rpy="0 0 0" />
       <geometry>
-        <mesh filename="package://rm_pioneer_description/meshes/standard_5/camera_base_link.STL" />
+        <mesh filename="package://rm_pioneer_description/meshes/standard5/camera_base_link.STL" />
       </geometry>
     </collision>
